File: Deauthentication_Injection.kicad_pcb (KiCad board)
At the start: 2 copper layers, 6 parts, among them J2 OLED, SW1 SW_Push, SW2 SW_Push, U1 ESP32-C3-DevKitM-1, U2 NRF24L01_Breakout

Commit message: Add files via upload
Parts:
- moved C1 62.5 mm to (55.5, 75.5), turned to 90 degrees
- moved U2 47.0 mm to (58.3, 59.1), turned to 180 degrees
- moved U1 31.4 mm to (90.9, 83.5), turned to 180 degrees
- moved SW1 23.9 mm to (118.5, 47.5)
- moved J2 22.3 mm to (107.0, 62.9), turned to -90 degrees
- moved SW2 18.0 mm to (118.8, 84.8)
Connections:
- U1 pad 2: Net-(U1-3V3-Pad2) -> +3.3V
- U1 pad 3: Net-(U1-3V3-Pad2) -> +3.3V
Routing:
- net VCC: track 0.00 -> 75.3 mm
- net /CE: track 0.00 -> 52.2 mm
- net GND: track 0.00 -> 52.2 mm
- net /SCL: track 0.00 -> 45.3 mm
- net /SDA: track 0.00 -> 43.2 mm
- net /MOSI: track 0.00 -> 36.2 mm
- net +3.3V: track 0.00 -> 22.4 mm
- net /MISO: track 0.00 -> 16.0 mm
- net /CSN: track 0.00 -> 15.1 mm
- net /IRQ: track 0.00 -> 14.0 mm
- net /SCK: track 0.00 -> 12.5 mm
