File: Deauthentication_Injection.kicad_sch (KiCad schematic)
At the start: 8 parts, among them J2 OLED, SW1 SW_Push, SW2 SW_Push, SW3 SW_Push, SW4 SW_Push, SW5 SW_Push, SW6 SW_Push, U1 ESP32-C3-DevKitM-1

Commit message: Add files via upload
Parts:
- removed SW3, SW4, SW5, SW6: SW_Push, Button_Switch_THT:SW_PUSH_6mm_H8.5mm, symbol Switch:SW_Push
- added C1: 1000, Capacitor_THT:CP_Radial_D14.0mm_P5.00mm, symbol Device:C
- added U2: NRF24L01_Breakout, RF_Module:nRF24L01_Breakout, symbol RF:NRF24L01_Breakout
Connections:
- net DOWN is gone; now on net SCL: U1.26 (IO9)
- net UP is gone; now on net SDA: U1.25 (IO8)
- net +3.3V: now also U1.2 (3V3), U1.3 (3V3)
- net GND: now also U1.1 (GND), U1.12 (GND), U1.15 (GND), U1.16 (GND), U1.19 (GND), U1.24 (GND), U1.27 (GND), U1.30 (GND), U1.6 (GND), U1.8 (GND), C1.1, U2.1 (GND)
- net SCL: no longer U1.20 (IO4)
- net SDA: no longer U1.21 (IO5)
- net VCC: now reaches U1.13 (5V), U1.14 (5V)
- net VCC: now also C1.2, U2.2 (VCC)
- net SW2: now reaches U1.4 (IO2)
- net SW2: now also SW2.1
- net SW1: now reaches U1.5 (IO3)
- net SW1: now also SW1.1
- net A renamed CE
- net CE: now also U2.3 (CE)
- net B renamed IRQ
- net IRQ: now also U2.8 (IRQ)
- net LEFT renamed CSN
- net CSN: now also U2.4 (~{CSN}); no longer SW1.1
- net RIGHT renamed MOSI
- net MOSI: now also U2.6 (MOSI); no longer SW2.1
- new net MISO: U1.20 (IO4), U2.7 (MISO)
- new net SCK: U1.21 (IO5), U2.5 (SCK)
Other:
- moved on the sheet: J2, SW1, SW2, U1
